Commit message: Feat: added a base differential drive robot with .urdf file

File: gen6s/test_diff_robot/urdf/test_diff_robot.urdf (robot description, URDF)
Before this commit: robot test_diff_robot, 4 links, 3 joints
Links:
- added link dummy_link
Joints:
- added joint dummy_joint: type fixed, parent dummy_link, child base_link
- joint left_wheel_joint: axis 0 0 1 -> 0 1 0
- joint right_wheel_joint: axis 0 0 -1 -> 0 1 0
