Commit message: Feat: minor fixees with plugins

File: gen6s/test_diff_robot/urdf/robots/test_diff_robot.urdf.xacro (robot description, xacro)
@@ -117,3 +117,13 @@
             <axis xyz="0 1 0"/>
         </joint>
+        <!-- Gazebo reference: -->
+        <gazebo reference="right_wheel">
+            <material>Gazebo/Blue</material>
+        </gazebo>
+        <gazebo reference="left_wheel">
+            <material>Gazebo/Blue</material>
+        </gazebo>
+        <gazebo reference="caster_wheel">
+            <material>Gazebo/Gray</material>
+        </gazebo>
     </robot>

Commit message: Fix:minor fixes to TF

File: gen6s/test_diff_robot/urdf/robots/test_diff_robot.urdf.xacro (robot description, xacro)
@@ -58,4 +58,9 @@
                 <material name="black"/>
             </visual>
+            <collision>
+                <geometry>
+                    <cylinder radius="0.05" length="0.02"/>
+                </geometry>
+            </collision>
             <inertial>
                 <mass value="0.5"/>
@@ -72,9 +77,17 @@
                 <material name="black"/>
             </visual>
-            <inertial>
+            <collision>
+                <geometry>
+                    <cylinder radius="0.05" length="0.02"/>
+                </geometry>
+            </collision>
+            <!-- <inertial>
                 <mass value="0.5"/>
                 <inertia ixx="0.01" ixy="0.0" ixz="0.0" iyy="0.01" iyz="0.0" izz="0.01"/>
                 <origin xyz="0 0 0" rpy="0 0 0"/>
-            </inertial>
+            </inertial> -->
+            <xacro:inertial_cylinder mass="0.5" length="0.02" radius="0.05">
+                <origin xyz="0 0 0" rpy="0 0 0"/>
+            </xacro:inertial_cylinder>
         </link>
         <!-- Caster Wheel -->
