Commit message: Fix: namespace error still persists but moving static from controllers.yaml, robot_launch.py

File: gen6s/test_diff_robot/urdf/robots/Ros2_control.xacro (robot description, xacro)
@@ -1,29 +1,34 @@
-<?xml version="1.0"?>
-<robot xmlns:xacro="http://www.ros.org/wiki/xacro">
-    <ros2_control name="GazeboSystem" type="system">
-        <hardware>
-            <plugin>gazebo_ros2_control/GazeboSystem</plugin>
-        </hardware>
-        <joint name="left_wheel_joint">
-            <command_interface name="velocity">
-                <param name="min">-10</param>
-                <param name="max">10</param>
-            </command_interface>
-            <state_interface name="velocity"/>
-            <state_interface name="position"/>
-        </joint>
-        <joint name="right_wheel_joint">
-            <command_interface name="velocity">
-                <param name="min">-10</param>
-                <param name="max">10</param>
-            </command_interface>
-            <state_interface name="velocity"/>
-            <state_interface name="position"/>
-        </joint>
-    </ros2_control>
-    <gazebo>
-        <plugin name="gazebo_ros2_control" filename="libgazebo_ros2_control.so">
-            <parameters>$(find articubot_one)/config/my_controllers.yaml</parameters>
-        </plugin>
-    </gazebo>
-</robot>
+    <?xml version="1.0"?>
+    <robot xmlns:xacro="http://www.ros.org/wiki/xacro">
+        <ros2_control name="GazeboSimSystem" type="system">
+            <hardware>
+                <plugin>gz_ros2_control/GazeboSimSystem</plugin>
+            </hardware>
+            <joint name="left_wheel_joint">
+                <command_interface name="velocity">
+                    <param name="min">-10</param>
+                    <param name="max">10</param>
+                </command_interface>
+                <state_interface name="velocity"/>
+                <state_interface name="position"/>
+            </joint>
+            <joint name="right_wheel_joint">
+                <command_interface name="velocity">
+                    <param name="min">-10</param>
+                    <param name="max">10</param>
+                </command_interface>
+                <state_interface name="velocity"/>
+                <state_interface name="position"/>
+            </joint>
+        </ros2_control>
+        <!-- <gazebo>
+            <plugin name="gazebo_ros2_control" filename="libgazebo_ros2_control.so">
+                <parameters>$(find test_diff_robot)/config/my_controllers.yaml</parameters>
+            </plugin>
+        </gazebo> -->
+        <gazebo>
+            <plugin filename="libgz_ros2_control-system.so" name="gz_ros2_control::GazeboSimROS2ControlPlugin">
+                <parameters>$(find test_diff_robot)/config/my_controllers.yaml</parameters>
+            </plugin>
+        </gazebo>
+    </robot>

File: gen6s/test_diff_robot/urdf/robots/gazebo_control.xacro (robot description, xacro)
@@ -6,5 +6,5 @@
             <left_joint>left_wheel_joint</left_joint>
             <right_joint>right_wheel_joint</right_joint>
-            <wheel_separation>0.35</wheel_separation>
+            <wheel_separation>0.3</wheel_separation>
             <wheel_diameter>0.1</wheel_diameter>
             <!-- Limits -->

File: gen6s/test_diff_robot/urdf/robots/inertial_macros.xacro (robot description, xacro)
@@ -1,5 +1,5 @@
 <?xml version="1.0"?>
 <robot xmlns:xacro="http://www.ros.org/wiki/xacro" >
-    <xacro:include filename="inertial_macros.xacro"/>
+    <!-- <xacro:include filename="inertial_macros.xacro"/> -->
     <!-- Specify some standard inertial calculations https://en.wikipedia.org/wiki/List_of_moments_of_inertia -->
     <!-- These make use of xacro's mathematical functionality -->

File: gen6s/test_diff_robot/urdf/robots/test_diff_robot.urdf copy.xacro (robot description, xacro)
@@ -1,4 +1,4 @@
 <?xml version="1.0"?>
-    <robot xmlns:xacro="http://wiki.ros.org/xacro" name="gen6s_diff">
+    <robot xmlns:xacro="http://wiki.ros.org/xacro">
     <!-- <xacro:property name="pi" value="3.141592653589793" /> -->
         <xacro:include filename="inertial_macros.xacro"/>
@@ -147,5 +147,3 @@
             <material>Gazebo/Gray</material>
         </gazebo>
-        <!-- <xacro:include filename="gazebo_control.xacro"/> -->
-        <xacro:include filename="Ros2_control.xacro"/>
     </robot>
