Commit message: Testing connection to gz sim from Ros2

File: gen6s/test_diff_robot/urdf/robots/expanded_robot_description.urdf (robot description, URDF)
Before this commit: robot gen6s_diff, 7 links, 6 joints
Links:
- removed link camera_link
- removed link camera_link_optical
- removed link caster_wheel
- removed link chassis
- link base_link: mass None -> 10; geometry collision box size=0.5 0.3 0.2; visual box size=0.5 0.3 0.2
- link left_wheel: mass 0.5 -> 1; geometry collision cylinder length=0.05 radius=0.1; visual cylinder length=0.05 radius=0.1
- link right_wheel: mass 0.5 -> 1; geometry collision cylinder length=0.05 radius=0.1; visual cylinder length=0.05 radius=0.1
Joints:
- removed joint camera_joint
- removed joint camera_optical_joint
- removed joint caster_wheel_joint
- removed joint chassis_joint
- joint left_wheel_joint: origin xyz=-0.2 0.15 0.05 rpy=1.57 0 0 -> xyz=0 0.15 0 rpy=1.57 0 0
- joint right_wheel_joint: origin xyz=-0.2 -0.15 0.05 rpy=1.57 0 0 -> xyz=0 -0.15 0 rpy=1.57 0 0

File: gen6s/test_diff_robot/urdf/robots/test_diff_robot.urdf.xacro (robot description, xacro)
@@ -67,12 +67,12 @@
                 </geometry>
             </collision>
-            <inertial>
+            <!-- <inertial>
                 <mass value="0.5"/>
                 <inertia ixx="0.01" ixy="0.0" ixz="0.0" iyy="0.01" iyz="0.0" izz="0.01"/>
                 <origin xyz="0 0 0" rpy="0 0 0"/>
-            </inertial>
-            <!-- <xacro:inertial_cylinder mass="0.5" length="0.02" radius="0.05">
+            </inertial> -->
+            <xacro:inertial_cylinder mass="0.5" length="0.02" radius="0.05">
                 <origin xyz="0 0 0" rpy="0 0 0"/>
-            </xacro:inertial_cylinder> -->
+            </xacro:inertial_cylinder>
         </link>
         <!-- Right Wheel -->
@@ -89,12 +89,12 @@
                 </geometry>
             </collision>
-            <inertial>
+            <!-- <inertial>
                 <mass value="0.5"/>
                 <inertia ixx="0.01" ixy="0.0" ixz="0.0" iyy="0.01" iyz="0.0" izz="0.01"/>
                 <origin xyz="0 0 0" rpy="0 0 0"/>
-            </inertial>
-            <!-- <xacro:inertial_cylinder mass="0.5" length="0.02" radius="0.05">
+            </inertial> -->
+            <xacro:inertial_cylinder mass="0.5" length="0.02" radius="0.05">
                 <origin xyz="0 0 0" rpy="0 0 0"/>
-            </xacro:inertial_cylinder> -->
+            </xacro:inertial_cylinder>
         </link>
         <!-- Caster Wheel -->
@@ -107,9 +107,12 @@
             </visual>
             <!-- add inertial for caster wheel -->
-            <inertial>
+            <!-- <inertial>
                 <mass value="0.5"/>
                 <inertia ixx="0.01" ixy="0.0" ixz="0.0" iyy="0.002" iyz="0.0" izz="0.002"/>
-                <origin xyz="0 0 0" rpy="0 0 0"/>
-            </inertial>
+                <origin xyz="0.1 0.0 0.5" rpy="0 0 0"/>
+            </inertial> -->
+            <xacro:inertial_sphere mass="0.5" radius="0.05">
+                <origin xyz="0.1 0 0.05"/>
+            </xacro:inertial_sphere>
         </link>
         <!-- Joints -->
@@ -132,5 +135,5 @@
             <axis xyz="0 1 0"/>
         </joint>
-        <joint name="caster_wheel_joint" type="fixed">
+        <joint name="caster_wheel_joint" type="continuous">
             <parent link="base_link"/>
             <child link="caster_wheel"/>
@@ -149,4 +152,14 @@
         </gazebo>
         <!-- <xacro:include filename="gazebo_control.xacro"/> -->
-        <xacro:include filename="ros2_control.xacro"/>
+        <!-- <xacro:include filename="ros2_control.xacro"/> -->
+        <plugin
+            filename="gz-sim-diff-drive-system"
+            name="gz::sim::systems::DiffDrive">
+            <left_joint>left_wheel_joint</left_joint>
+            <right_joint>right_wheel_joint</right_joint>
+            <wheel_separation>0.3</wheel_separation>
+            <wheel_radius>0.05</wheel_radius>
+            <odom_publish_frequency>1</odom_publish_frequency>
+            <topic>cmd_vel</topic>
+        </plugin>
     </robot>

Commit message: tryinhg to fix the movement of the bot with adino urdf

File: gen6s/test_diff_robot/urdf/robots/expanded_robot_description.urdf (robot description, URDF)
Before this commit: robot diff_drive_robot, 3 links, 2 joints
Links:
- added link base_footprint
- added link caster_wheel, mass 0.01; collision sphere radius=0.01; visual sphere radius=0.01
- added link chassis, mass 0.5; collision box size=0.335 0.265 0.138; visual box size=0.335 0.265 0.138
- link base_link: mass 10 -> None; geometry 
- link left_wheel: mass 1 -> 0.05; geometry collision sphere radius=0.033; visual cylinder length=0.026 radius=0.033
- link right_wheel: mass 1 -> 0.05; geometry collision sphere radius=0.033; visual cylinder length=0.026 radius=0.033
Joints:
- added joint base_footprint_joint: type fixed, parent base_link, child base_footprint, origin xyz=0 0 0.069 rpy=0 0 0
- added joint caster_wheel_joint: type fixed, parent chassis, child caster_wheel, origin xyz=0.075 0 -0.013
- added joint chassis_joint: type fixed, parent base_link, child chassis, origin xyz=-0.226 0 -0.01
- joint left_wheel_joint: axis 0 1 0 -> 0 0 1; origin xyz=0 0.15 0 rpy=1.57 0 0 -> xyz=0 0.1485 0 rpy=-1.5707963267948966 0 0
- joint right_wheel_joint: axis 0 1 0 -> 0 0 -1; origin xyz=0 -0.15 0 rpy=1.57 0 0 -> xyz=0 -0.1485 0 rpy=1.5707963267948966 0 0

File: gen6s/test_diff_robot/urdf/robots/test_diff_robot.urdf.xacro (robot description, xacro)
@@ -32,4 +32,10 @@
         </link> -->
         <link name="base_link">
+            <collision>
+                <origin xyz="0 0 ${height1/2}" rpy="0 0 0"/>
+                <geometry>
+                <box size="${width} ${width} ${height1}"/>
+                </geometry>
+            </collision>
         </link>
         <!-- CHASSIS LINK -->

Commit message: modified xacro and launch

File: gen6s/test_diff_robot/urdf/robots/expanded_robot_description.urdf (robot description, URDF)
Before this commit: robot andino, 6 links, 5 joints
Joints:
- joint base_footprint_joint: origin xyz=0 0 0.069 rpy=0 0 0 -> xyz=0 0 0 rpy=0 0 0
